Commit message: Updated blending_eff_macro.xacro to use the calibration macro

File: godel_robot_config/urdf/asus_sensor_macro.xacro (robot description, xacro)
@@ -1,4 +1,5 @@
 <?xml version="1.0" ?>
 <robot name="asus_sensor" xmlns:xacro="http://ros.org/wiki/xacro">
+	<xacro:include filename="$(find godel_robot_config)/urdf/calibration_transform.xacro"/>
 	<xacro:property name="asus_length" value="0.220"/>
 	<xacro:property name="asus_width" value="0.040"/>
@@ -79,4 +80,6 @@
 			<origin xyz="${x_val} ${y_val} ${z_val}" rpy="${roll} ${pitch} ${yaw}"/>
 		</joint>
+                             <!-- Replace the fixed joint destined for calibration by the calibration definition -->
+		<xacro:macro name="calibration_definition" params="${prefix}asus_link ${parent_link} ${x_val} ${y_val} ${z_val} ${roll} ${pitch} ${yaw}">
 		<!-- end of world joints -->
 	</xacro:macro>

File: godel_robot_config/urdf/blending_eff_macro.xacro (robot description, xacro)
@@ -1,5 +1,5 @@
 <?xml version="1.0" ?>
 <robot xmlns:xacro="http://ros.org/wiki/xacro">
-	<xacro:include filename="$(find godel_robot_config)/urdf/asus_sensor_macro.xacro"/>
+	<xacro:include filename="$(find godel_robot_config)/urdf/asus_sensor_cal_macro.xacro"/>
 	<!-- parameter list -->
 	<xacro:property name="gripper_length" value="0.0"/>
@@ -29,6 +29,5 @@
 			<link name="${prefix}tcp_frame"/>
 			<link name="${prefix}asus_mount"/>
-		<xacro:asus_sensor_definitions prefix="${prefix}" parent_link="${prefix}asus_mount"
-				x_val="0" y_val="0" z_val="0" roll="3.14" pitch="0.0" yaw="0.0"/>
+		<xacro:asus_sensor_definitions prefix="${prefix}" parent_link="${prefix}asus_mount" />
 		<!-- joint definitions -->
 			<joint name="${prefix}gripper_to_palm" type="fixed">
