Commit message: Added files and modifications to allow extrinsic calibration

File: godel_robot_config/urdf/asus_sensor_cal_macro.xacro (robot description, xacro)
@@ -56,5 +56,5 @@
 			<parent link="${prefix}asus_frame"/>
 			<child link="${prefix}asus_ir_link"/>
-			<origin rpy="0 0 0" xyz="0 0 0"/>
+			<origin rpy="0 0 0" xyz="0 0.0476 0"/>
 		</joint>
 		<joint name="${prefix}asus_ir_optical_frame_joint" type="fixed">
@@ -66,5 +66,5 @@
 			<parent link="${prefix}asus_ir_link"/>
 			<child link="${prefix}asus_rgb_link"/>
-			<origin rpy="0 0 0" xyz="0 -0.03 0"/>
+			<origin rpy="0 0 0" xyz="0 -0.025 0"/>
 		</joint>
 		<joint name="${prefix}asus_rgb_optical_frame_joint" type="fixed">

File: godel_robot_config/urdf/sia20d_workspace_calibrate.xacro (robot description, xacro)
@@ -22,4 +22,16 @@
 		</collision>
 	</link>
+                   <link name="zcirclegrid7x5">
+                          <visual>
+                                <geometry>
+                                    <mesh filename="package://godel_robot_config/meshes/circlegrid_wcolor.dae" />
+                                </geometry>
+                           </visual>
+                           <collision>
+                                   <geometry>
+                                          <box size=".001 .001 .001" />
+                                  </geometry>
+                            </collision>
+	</link>
 	<!-- instantiating sensor definitions -->
 	<xacro:sensor_definitions prefix="${arm_prefix}" parent_link="${arm_prefix}base_link"
@@ -34,4 +46,12 @@
 		<origin xyz="0 ${coupler_height} 0" rpy="0.0 0.0 0.0"/>
 	</joint>
+	<!-- REPLACE WITH A CALIBRATABLE TRANSFORM -->
+	<!-- joint name="ref2target" type="fixed">
+		<parent link="world_frame"/>
+		<child link="circlegrid7x5"/>
+		<origin xyz="0.85 -0.2 0.0" rpy="0.0 0.0 3.1415"/>
+	</joint-->
+	<xacro:include filename="$(find godel_robot_config)/urdf/calibration_transform.xacro"/>
+	<xacro:calibration_definitions child_link="zcirclegrid7x5" parent_link="world_frame" />
 	<!-- start of arm-workcell joint definitions -->
 	<joint name="world_to_base" type="fixed">
